Commit message: Second commit

File: ros2_ws/install/gazebo_hello/share/gazebo_hello/urdf/pan_tilt.urdf.xacro (robot description, xacro)
@@ -7,5 +7,5 @@
     <!-- Fixed joint from world to base_link (like the example) -->
     <joint name="base_joint" type="fixed">
-        <origin xyz="1.5 1.0 0" rpy="0 0 0"/>
+        <origin xyz="0 0 0" rpy="0 0 0"/>
         <parent link="world"/>
         <child link="base_link"/>
@@ -62,5 +62,5 @@
     </link>
     <!-- Pan Joint -->
-    <joint name="pan_joint" type="revolute">
+    <joint name="pan_joint" type="continuous">
         <parent link="base_link"/>
         <child link="pan_link"/>

Commit message: camera working

File: ros2_ws/install/gazebo_hello/share/gazebo_hello/urdf/pan_tilt.urdf.xacro (robot description, xacro)
@@ -3,4 +3,5 @@
     <!-- Include common materials and inertial macros -->
     <xacro:include filename="example_include.xacro" />
+    <xacro:include filename="camera.xacro" />
     <!-- Empty world link -->
     <link name="world"></link>
@@ -95,4 +96,5 @@
     <!-- Tilt Joint -->
     <joint name="tilt_joint" type="revolute">
+        <gravity>false</gravity>
         <parent link="pan_link"/>
         <child link="tilt_link"/>
@@ -102,33 +104,4 @@
         <dynamics damping="0.5" friction="0.1"/>
     </joint>
-    <!-- Camera Link -->
-    <link name="camera_link">
-        <visual>
-            <origin xyz="0 0 0" rpy="0 0 0"/>
-            <geometry>
-                <box size="0.03 0.04 0.02"/>
-            </geometry>
-            <material name="black">
-                <color rgba="0.1 0.1 0.1 1"/>
-            </material>
-        </visual>
-        <collision>
-            <origin xyz="0 0 0" rpy="0 0 0"/>
-            <geometry>
-                <box size="0.03 0.04 0.02"/>
-            </geometry>
-        </collision>
-        <inertial>
-            <origin xyz="0 0 0" rpy="0 0 0"/>
-            <mass value="0.1"/>
-            <inertia ixx="0.000003" ixy="0" ixz="0" iyy="0.000003" iyz="0" izz="0.000004"/>
-        </inertial>
-    </link>
-    <!-- Fixed Camera Joint -->
-    <joint name="camera_joint" type="fixed">
-        <parent link="tilt_link"/>
-        <child link="camera_link"/>
-        <origin xyz="0.06 0 0" rpy="0 0 0"/>
-    </joint>
     <!-- Gazebo-specific stuff (materials, plugins, depth camera, etc.) -->
     <xacro:include filename="example_gazebo.xacro" />
